File: splanck throughhole.kicad_pcb (KiCad board)
At the start: 2 copper layers, 106.7 x 73.7 mm, 51 parts, among them K1 XLR3, SW1 SW_PUSH, SW10 SW_PUSH, SW11 SW_PUSH, SW12 SW_PUSH, SW13 SW_PUSH, SW14 SW_PUSH, SW15 SW_PUSH, SW16 SW_PUSH, SW17 SW_PUSH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

Commit message: brought the pcb up to date and fixed reset pin
Parts:
- removed SW25: SW_PUSH, Buttons_Switches_SMD:SW_SPST_FSMSM
- added extra data line: TEST_1P, Wire_Pads:SolderWirePad_single_0-8mmDrill, F.Cu at (135.0, 50.0)
- moved D2 9.11 mm to (49.0, 61.2), turned to 270 degrees
- moved D4 9.09 mm to (48.8, 98.8), turned to 270 degrees
- moved D3 8.98 mm to (48.8, 80.0), turned to 270 degrees
- moved D21 4.20 mm to (128.0, 49.3)
- moved D1 3.84 mm to (41.1, 49.5)
- moved D6 3.44 mm to (59.9, 70.1)
Connections:
- D10 pad 2: Net-(D10-Pad2) -> row1
- D14 pad 2: Net-(D10-Pad2) -> row1
- D18 pad 2: Net-(D10-Pad2) -> row1
- D2 pad 2: Net-(D10-Pad2) -> row1
- D22 pad 2: Net-(D10-Pad2) -> row1
- D6 pad 2: Net-(D10-Pad2) -> row1
- K1 pad 4: (no net) -> Net-(K1-Pad4)
- U1 pad 23: data -> Net-(U1-Pad23)
- U1 pad 24: Net-(U1-Pad24) -> data
- U1 pad 27: GND -> Net-(U1-Pad27)
- U1 pad 28: Net-(U1-Pad28) -> GND
- U1 pad 3: Net-(SW25-Pad1) -> GND
Routing:
- net row1: track 0.00 -> 98.3 mm, vias 0 -> 1
- net Net-(D10-Pad2): track 85.1 -> 0.00 mm
- net GND: track 0.00 -> 39.1 mm, vias 0 -> 3
- net Net-(U1-Pad2): track 25.7 -> 0.00 mm
- net Net-(K1-Pad4): track 0.00 -> 20.4 mm
- net Net-(SW25-Pad1): track 18.8 -> 0.00 mm
- net Net-(D4-Pad1): track 7.62 -> 19.7 mm
- net Net-(D2-Pad1): track 7.62 -> 12.3 mm
- net Net-(D3-Pad1): track 7.62 -> 11.9 mm
- net row2: track 112.2 -> 107.9 mm
- net Net-(D21-Pad1): track 6.98 -> 11.3 mm
- net row3: track 135.9 -> 131.7 mm
- net row0: track 101.5 -> 105.6 mm
- net Net-(D1-Pad1): track 7.62 -> 11.6 mm
- net Net-(D6-Pad1): track 11.1 -> 14.8 mm, vias 1 -> 2
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Other:
- board size 106.7 x 73.7 mm -> 106.7 x 72.4 mm
- board text added: "1. header pins 2. switches 3.pro micro"
- board text added: "Designed by Wootpatoot for all the cheap makers"
- board text removed: "designed by Max aka wootpatoot"
- board text removed: "header pins first dingus"
